Commit message: update

File: src/panda_simulation/franka_description/robots/panda_arm.xacro (robot description, xacro)
@@ -11,4 +11,5 @@
   <xacro:property name="mass_link7" value="0.45606" />
   <xacro:property name="mass_link8" value="0.001" />
+  <xacro:property name="mass_marker" value="0.00001" />
   <!-- Wrong masses to test adaptability of the algorithms, on purpose off by 20% -->
   <!--xacro:property name="mass_link0" value="3.66357" />
@@ -252,4 +253,18 @@
       <dynamics damping="${joint_damping}"/>
     </joint>
+<!-- ADD MARKER TO LAST JOINT -->
+    <link name="${arm_id}_marker">
+      <visual>
+        <origin xyz="0 0 0" rpy="0 0 0" />
+        <geometry>
+          <mesh filename="package://${description_pkg}/meshes/aruco_marker.dae"/>
+        </geometry>
+      </visual>
+    </link>
+    <joint name="robot_to_marker" type="fixed">
+      <parent link="${arm_id}_link7" />
+      <child link="${arm_id}_marker" />
+    <origin xyz="0.05 0.0 0.0" rpy="0.0 1.57 0.0" />
+    </joint>
     <link name="${arm_id}_link8">
       <inertial>
@@ -263,4 +278,5 @@
       <parent link="${arm_id}_link7"/>
       <child link="${arm_id}_link8"/>
+      <child link="${arm_id}_marker"/>
       <axis xyz="0 0 1"/>
       <limit effort="1" lower="0" upper="0.1" velocity="0.1"/>
